File: schematics/rev2/Matrix.kicad_sch (KiCad schematic)
At the start: 94 parts, among them SW1 KS-33, SW10 KS-33, SW11 KS-33, SW12 KS-33, SW13 KS-33, SW14 KS-33, SW15 KS-33, SW16 KS-33, SW17 KS-33, SW18 KS-33, SW19 KS-33, SW2 KS-33, SW20 KS-33, SW21 KS-33, SW22 KS-33, SW23 KS-33, SW24 KS-33, SW25 KS-33, SW26 KS-33, SW27 KS-33, SW28 KS-33, SW29 KS-33, SW3 KS-33, SW30 KS-33, SW31 KS-33, SW32 KS-33, SW33 KS-33, SW34 KS-33, SW35 KS-33, SW36 KS-33, SW37 KS-33, SW38 KS-33, SW39 KS-33, SW4 KS-33, SW40 KS-33, SW41 KS-33, SW42 KS-33, SW43 KS-33, SW44 KS-33, SW45 KS-33, SW46 KS-33, SW48 KS-33, SW5 KS-33, SW6 KS-33, SW7 KS-33, SW8 KS-33, SW9 KS-33

Commit message: Update key layout, increase debounce, PCB update
Parts:
- SW1, SW10, SW11, SW12, SW13, SW14, SW15, SW16, SW17, SW18, SW19, SW2, SW20, SW21, SW22, SW23, SW24, SW25, SW26, SW27, SW28, SW29, SW3, SW30, SW31, SW32, SW33, SW34, SW35, SW36, SW37, SW38, SW39, SW4, SW40, SW41, SW42, SW43, SW44, SW45, SW46, SW48, SW5, SW6, SW7, SW8, SW9: footprint Keyboard Switches:SW_Gateron_LowProfile_THT -> Library:Cherry MX switch
Changed lines of the file:
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@@
 			)
 		)
-		(property "Footprint" "Keyboard Switches:SW_Gateron_LowProfile_THT"
+		(property "Footprint" "Library:Cherry MX switch"
 			(at 78.74 139.7 0)
 			(effects
@@
 			)
 		)
-		(property "Footprint" "Keyboard Switches:SW_Gateron_LowProfile_THT"
+		(property "Footprint" "Library:Cherry MX switch"
 			(at 162.56 118.11 0)
 			(effects
@@
 			)
 		)
-		(property "Footprint" "Keyboard Switches:SW_Gateron_LowProfile_THT"
+		(property "Footprint" "Library:Cherry MX switch"
 			(at 179.07 99.06 0)
 			(effects
@@
 			)
 		)
-		(property "Footprint" "Keyboard Switches:SW_Gateron_LowProfile_THT"
+		(property "Footprint" "Library:Cherry MX switch"
 			(at 210.82 118.11 0)
 			(effects
@@
 			)
 		)
-		(property "Footprint" "Keyboard Switches:SW_Gateron_LowProfile_THT"
+		(property "Footprint" "Library:Cherry MX switch"
 			(at 115.57 99.06 0)
 			(effects
@@
 			)
 		)
-		(property "Footprint" "Keyboard Switches:SW_Gateron_LowProfile_THT"
+		(property "Footprint" "Library:Cherry MX switch"
 			(at 227.33 99.06 0)
 			(effects
@@
 			)
 		)
-		(property "Footprint" "Keyboard Switches:SW_Gateron_LowProfile_THT"
+		(property "Footprint" "Library:Cherry MX switch"
 			(at 179.07 81.28 0)
 			(effects
@@
 			)
 		)
-		(property "Footprint" "Keyboard Switches:SW_Gateron_LowProfile_THT"
+		(property "Footprint" "Library:Cherry MX switch"
 			(at 210.82 139.7 0)
 			(effects
@@
 			)
 		)
-		(property "Footprint" "Keyboard Switches:SW_Gateron_LowProfile_THT"
+		(property "Footprint" "Library:Cherry MX switch"
 			(at 52.07 99.06 0)
 			(effects
@@
 			)
 		)
-		(property "Footprint" "Keyboard Switches:SW_Gateron_LowProfile_THT"
+		(property "Footprint" "Library:Cherry MX switch"
 			(at 97.79 99.06 0)
 			(effects
@@
 			)
 		)
-		(property "Footprint" "Keyboard Switches:SW_Gateron_LowProfile_THT"
+		(property "Footprint" "Library:Cherry MX switch"
 			(at 179.07 139.7 0)
 			(effects
@@
 			)
 		)
-		(property "Footprint" "Keyboard Switches:SW_Gateron_LowProfile_THT"
+		(property "Footprint" "Library:Cherry MX switch"
 			(at 194.31 81.28 0)
 			(effects
@@
 			)
 		)
-		(property "Footprint" "Keyboard Switches:SW_Gateron_LowProfile_THT"
+		(property "Footprint" "Library:Cherry MX switch"
 			(at 80.01 118.11 0)
 			(effects
@@
 			)
 		)
-		(property "Footprint" "Keyboard Switches:SW_Gateron_LowProfile_THT"
+		(property "Footprint" "Library:Cherry MX switch"
 			(at 52.07 118.11 0)
 			(effects
@@
 			)
 		)
-		(property "Footprint" "Keyboard Switches:SW_Gateron_LowProfile_THT"
+		(property "Footprint" "Library:Cherry MX switch"
 			(at 195.58 139.7 0)
 			(effects
@@
 			)
 		)
-		(property "Footprint" "Keyboard Switches:SW_Gateron_LowProfile_THT"
+		(property "Footprint" "Library:Cherry MX switch"
 			(at 227.33 81.28 0)
 			(effects
@@
 			)
 		)
-		(property "Footprint" "Keyboard Switches:SW_Gateron_LowProfile_THT"
+		(property "Footprint" "Library:Cherry MX switch"
 			(at 242.57 81.28 0)
 			(effects
@@
 			)
 		)
-		(property "Footprint" "Keyboard Switches:SW_Gateron_LowProfile_THT"
+		(property "Footprint" "Library:Cherry MX switch"
 			(at 194.31 118.11 0)
 			(effects
@@
 			)
 		)
-		(property "Footprint" "Keyboard Switches:SW_Gateron_LowProfile_THT"
+		(property "Footprint" "Library:Cherry MX switch"
 			(at 130.81 118.11 0)
 			(effects
@@
 			)
 		)
-		(property "Footprint" "Keyboard Switches:SW_Gateron_LowProfile_THT"
+		(property "Footprint" "Library:Cherry MX switch"
 			(at 52.07 81.28 0)
 			(effects
@@
 			)
 		)
-		(property "Footprint" "Keyboard Switches:SW_Gateron_LowProfile_THT"
+		(property "Footprint" "Library:Cherry MX switch"
 			(at 162.56 81.28 0)
 			(effects
@@
 			)
 		)
-		(property "Footprint" "Keyboard Switches:SW_Gateron_LowProfile_THT"
+		(property "Footprint" "Library:Cherry MX switch"
 			(at 194.31 99.06 0)
 			(effects
@@
 			)
 		)
-		(property "Footprint" "Keyboard Switches:SW_Gateron_LowProfile_THT"
+		(property "Footprint" "Library:Cherry MX switch"
 			(at 242.57 99.06 0)
 			(effects
@@
 			)
 		)
-		(property "Footprint" "Keyboard Switches:SW_Gateron_LowProfile_THT"
+		(property "Footprint" "Library:Cherry MX switch"
 			(at 147.32 81.28 0)
 			(effects
@@
 			)
 		)
-		(property "Footprint" "Keyboard Switches:SW_Gateron_LowProfile_THT"
+		(property "Footprint" "Library:Cherry MX switch"
 			(at 115.57 139.7 0)
 			(effects
@@
 			)
 		)
-		(property "Footprint" "Keyboard Switches:SW_Gateron_LowProfile_THT"
+		(property "Footprint" "Library:Cherry MX switch"
 			(at 210.82 99.06 0)
 			(effects
@@
 			)
 		)
-		(property "Footprint" "Keyboard Switches:SW_Gateron_LowProfile_THT"
+		(property "Footprint" "Library:Cherry MX switch"
 			(at 147.32 99.06 0)
 			(effects
@@
 			)
 		)
-		(property "Footprint" "Keyboard Switches:SW_Gateron_LowProfile_THT"
+		(property "Footprint" "Library:Cherry MX switch"
 			(at 115.57 118.11 0)
 			(effects
@@
 			)
 		)
-		(property "Footprint" "Keyboard Switches:SW_Gateron_LowProfile_THT"
+		(property "Footprint" "Library:Cherry MX switch"
 			(at 130.81 99.06 0)
 			(effects
@@
 			)
 		)
-		(property "Footprint" "Keyboard Switches:SW_Gateron_LowProfile_THT"
+		(property "Footprint" "Library:Cherry MX switch"
 			(at 115.57 81.28 0)
 			(effects
@@
 			)
 		)
-		(property "Footprint" "Keyboard Switches:SW_Gateron_LowProfile_THT"
+		(property "Footprint" "Library:Cherry MX switch"
 			(at 97.79 118.11 0)
 			(effects
@@
 			)
 		)
-		(property "Footprint" "Keyboard Switches:SW_Gateron_LowProfile_THT"
+		(property "Footprint" "Library:Cherry MX switch"
 			(at 52.07 139.7 0)
 			(effects
@@
 			)
 		)
-		(property "Footprint" "Keyboard Switches:SW_Gateron_LowProfile_THT"
+		(property "Footprint" "Library:Cherry MX switch"
 			(at 179.07 118.11 0)
 			(effects
@@
 			)
 		)
-		(property "Footprint" "Keyboard Switches:SW_Gateron_LowProfile_THT"
+		(property "Footprint" "Library:Cherry MX switch"
 			(at 78.74 99.06 0)
 			(effects
@@
 			)
 		)
-		(property "Footprint" "Keyboard Switches:SW_Gateron_LowProfile_THT"
+		(property "Footprint" "Library:Cherry MX switch"
 			(at 242.57 139.7 0)
 			(effects
@@
 			)
 		)
-		(property "Footprint" "Keyboard Switches:SW_Gateron_LowProfile_THT"
+		(property "Footprint" "Library:Cherry MX switch"
 			(at 147.32 118.11 0)
 			(effects
@@
 			)
 		)
-		(property "Footprint" "Keyboard Switches:SW_Gateron_LowProfile_THT"
+		(property "Footprint" "Library:Cherry MX switch"
 			(at 130.81 81.28 0)
 			(effects
@@
 			)
 		)
-		(property "Footprint" "Keyboard Switches:SW_Gateron_LowProfile_THT"
+		(property "Footprint" "Library:Cherry MX switch"
 			(at 162.56 139.7 0)
 			(effects
@@
 			)
 		)
-		(property "Footprint" "Keyboard Switches:SW_Gateron_LowProfile_THT"
+		(property "Footprint" "Library:Cherry MX switch"
 			(at 97.79 81.28 0)
 			(effects
@@
 			)
 		)
-		(property "Footprint" "Keyboard Switches:SW_Gateron_LowProfile_THT"
+		(property "Footprint" "Library:Cherry MX switch"
 			(at 162.56 99.06 0)
 			(effects
@@
 			)
 		)
-		(property "Footprint" "Keyboard Switches:SW_Gateron_LowProfile_THT"
+		(property "Footprint" "Library:Cherry MX switch"
 			(at 78.74 81.28 0)
 			(effects
@@
 			)
 		)
-		(property "Footprint" "Keyboard Switches:SW_Gateron_LowProfile_THT"
+		(property "Footprint" "Library:Cherry MX switch"
 			(at 242.57 118.11 0)
 			(effects
@@
 			)
 		)
-		(property "Footprint" "Keyboard Switches:SW_Gateron_LowProfile_THT"
+		(property "Footprint" "Library:Cherry MX switch"
 			(at 226.06 139.7 0)
 			(effects
@@
 			)
 		)
-		(property "Footprint" "Keyboard Switches:SW_Gateron_LowProfile_THT"
+		(property "Footprint" "Library:Cherry MX switch"
 			(at 210.82 81.28 0)
 			(effects
@@
 			)
 		)
-		(property "Footprint" "Keyboard Switches:SW_Gateron_LowProfile_THT"
+		(property "Footprint" "Library:Cherry MX switch"
 			(at 130.81 139.7 0)
 			(effects
@@
 			)
 		)
-		(property "Footprint" "Keyboard Switches:SW_Gateron_LowProfile_THT"
+		(property "Footprint" "Library:Cherry MX switch"
 			(at 97.79 139.7 0)
 			(effects
@@
 			)
 		)
-		(property "Footprint" "Keyboard Switches:SW_Gateron_LowProfile_THT"
+		(property "Footprint" "Library:Cherry MX switch"
 			(at 227.33 118.11 0)
 			(effects
