File: schematics/rev2/40 Keyboard.kicad_pcb (KiCad board)
At the start: 2 copper layers, 247 x 100.8 mm, 109 parts, among them J2 2171790001, SW1 KS-33, SW10 KS-33, SW11 KS-33, SW12 KS-33, SW13 KS-33, SW14 KS-33, SW15 KS-33, SW16 KS-33, SW17 KS-33, SW18 KS-33, SW19 KS-33, SW2 KS-33, SW20 KS-33, SW21 KS-33, SW22 KS-33, SW23 KS-33, SW24 KS-33, SW25 KS-33, SW26 KS-33, SW27 KS-33, SW28 KS-33, SW29 KS-33, SW3 KS-33, SW30 KS-33, SW31 KS-33, SW32 KS-33, SW33 KS-33, SW34 KS-33, SW35 KS-33, SW36 KS-33, SW37 KS-33, SW38 KS-33, SW39 KS-33, SW4 KS-33, SW40 KS-33, SW41 KS-33, SW42 KS-33, SW43 KS-33, SW44 KS-33, SW45 KS-33, SW46 KS-33, SW47 RESET, SW48 KS-33, SW5 KS-33, SW6 KS-33, SW7 KS-33, SW8 KS-33, SW9 KS-33, U2 ATMEGA32U4-AU, Y1 16Mhz

Commit message: Update key layout, increase debounce, PCB update
Parts:
- removed C1: C3216X7R2A334K130AA, Capacitor_SMD:C_1206_3216Metric
- removed D48: LED, LED_THT:LED_D3.0mm
- removed R15: 1k, Resistor_SMD:R_1206_3216Metric
- added SW49: HWB, Jumper:SolderJumper-2_P1.3mm_Open_Pad1.0x1.5mm, B.Cu at (185.1, 59.2)
- added U1: ~, Connector_PinHeader_2.54mm:PinHeader_2x03_P2.54mm_Vertical, B.Cu at (197.0, 59.2)
- SW1, SW10, SW11, SW12, SW13, SW14, SW15, SW16, SW17, SW18, SW19, SW2, SW20, SW21, SW22, SW23, SW24, SW25, SW26, SW27, SW28, SW29, SW3, SW30, SW31, SW32, SW33, SW34, SW35, SW36, SW37, SW38, SW39, SW4, SW40, SW41, SW42, SW43, SW44, SW45, SW46, SW48, SW5, SW6, SW7, SW8, SW9: footprint Keyboard Switches:SW_Gateron_LowProfile_THT -> Library:Cherry MX switch
- moved SW47 72.4 mm to (188.1, 59.2), turned to 90 degrees
- moved C6 70.9 mm to (183.2, 64.7), turned to 0 degrees
- moved Y1 61.2 mm to (188.2, 68.7), turned to 0 degrees
- moved C5 51.7 mm to (194.1, 64.6), turned to 180 degrees
- moved J2 40.0 mm to (168.1, 57.1)
- moved R18 39.6 mm to (161.0, 59.1)
- moved R19 39.3 mm to (158.0, 59.1)
- moved C7 37.2 mm to (202.3, 62.2)
- moved R16 37.2 mm to (202.4, 67.4)
- moved R17 37.2 mm to (202.4, 64.9)
- moved U2 35.8 mm to (214.2, 62.6), turned to 180 degrees
- moved C2 35.6 mm to (152.7, 59.1), turned to 90 degrees
- moved SW42 5.65 mm to (187.6, 130.2)
- moved SW43 5.65 mm to (159.1, 130.2)
- moved SW45 5.65 mm to (232.7, 129.9)
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Connections:
- net /Microcontroller/RSET renamed RSET
- U2 pad 10: COL_6 -> MOSI
- U2 pad 11: COL_5 -> MISO
- U2 pad 12: /Microcontroller/RTS -> COL_12
- U2 pad 18: COL_11 -> COL_1
- U2 pad 19: COL_12 -> COL_2
- U2 pad 20: /Microcontroller/32U4_RX -> COL_3
- U2 pad 21: /Microcontroller/32U4_TX -> COL_4
- U2 pad 22: /Microcontroller/CTS -> COL_6
- U2 pad 25: unconnected-(U2-PD4-Pad25) -> COL_5
- U2 pad 26: unconnected-(U2-PD6-Pad26) -> COL_7
- U2 pad 27: unconnected-(U2-PD7-Pad27) -> COL_8
- U2 pad 28: COL_4 -> COL_9
- U2 pad 29: COL_3 -> COL_10
- U2 pad 30: COL_2 -> COL_11
- U2 pad 31: COL_9 -> unconnected-(U2-PC6-Pad31)
- U2 pad 32: COL_10 -> unconnected-(U2-PC7-Pad32)
- U2 pad 33: /Microcontroller/32U4_HWB -> Net-(U2-PE2)
- U2 pad 37: COL_1 -> unconnected-(U2-PF6-Pad37)
- U2 pad 8: COL_8 -> unconnected-(U2-PB0-Pad8)
- U2 pad 9: COL_7 -> SCK
Routing:
- removed copper zone on F.Cu, net GND
Other:
- board size 247 x 100.8 mm -> 247 x 91.2 mm
- board text added: "${REFERENCE}"
- board text added: "Designed by Luke Zambella Rev2"
- board text removed: "Designed by Luke Zambella"

Commit message: Update schematic and board layout
Parts:
- removed J2: 2171790001, Library:MOLEX_2171790001
- removed SW47: RESET, Jumper:SolderJumper-2_P1.3mm_Open_Pad1.0x1.5mm
- removed SW49: HWB, Jumper:SolderJumper-2_P1.3mm_Open_Pad1.0x1.5mm
- added D1: D, Diode_SMD:D_SOD-123, B.Cu at (250.1, 128.2)
- added D48: LED, LED_SMD:LED_1206_3216Metric_Pad1.42x1.75mm_HandSolder, F.Cu at (25.9, 82.5)
- added D49: LED, LED_SMD:LED_1206_3216Metric_Pad1.42x1.75mm_HandSolder, F.Cu at (44.9, 82.5)
- added D51: LED, LED_SMD:LED_1206_3216Metric_Pad1.42x1.75mm_HandSolder, F.Cu at (64.0, 82.6)
- added D52: LED, LED_SMD:LED_1206_3216Metric_Pad1.42x1.75mm_HandSolder, F.Cu at (83.0, 82.6)
- added D53: LED, LED_SMD:LED_1206_3216Metric_Pad1.42x1.75mm_HandSolder, F.Cu at (101.9, 82.5)
- added D54: LED, LED_SMD:LED_1206_3216Metric_Pad1.42x1.75mm_HandSolder, F.Cu at (120.9, 82.5)
- added D55: LED, LED_SMD:LED_1206_3216Metric_Pad1.42x1.75mm_HandSolder, F.Cu at (140.0, 82.6)
- added D56: LED, LED_SMD:LED_1206_3216Metric_Pad1.42x1.75mm_HandSolder, F.Cu at (159.0, 82.6)
- added D57: LED, LED_SMD:LED_1206_3216Metric_Pad1.42x1.75mm_HandSolder, F.Cu at (178.0, 82.6)
- added D58: LED, LED_SMD:LED_1206_3216Metric_Pad1.42x1.75mm_HandSolder, F.Cu at (197.0, 82.6)
- added D59: LED, LED_SMD:LED_1206_3216Metric_Pad1.42x1.75mm_HandSolder, F.Cu at (216.1, 82.6)
- added D60: LED, LED_SMD:LED_1206_3216Metric_Pad1.42x1.75mm_HandSolder, F.Cu at (234.9, 82.6)
- added D61: LED, LED_SMD:LED_1206_3216Metric_Pad1.42x1.75mm_HandSolder, F.Cu at (254.0, 82.6)
- added D62: LED, LED_SMD:LED_1206_3216Metric_Pad1.42x1.75mm_HandSolder, F.Cu at (27.9, 101.6)
- added D63: LED, LED_SMD:LED_1206_3216Metric_Pad1.42x1.75mm_HandSolder, F.Cu at (49.8, 101.6)
- added D64: LED, LED_SMD:LED_1206_3216Metric_Pad1.42x1.75mm_HandSolder, F.Cu at (68.6, 101.6)
- added D65: LED, LED_SMD:LED_1206_3216Metric_Pad1.42x1.75mm_HandSolder, F.Cu at (87.7, 101.6)
- added D66: LED, LED_SMD:LED_1206_3216Metric_Pad1.42x1.75mm_HandSolder, F.Cu at (106.6, 101.6)
- added D67: LED, LED_SMD:LED_1206_3216Metric_Pad1.42x1.75mm_HandSolder, F.Cu at (125.9, 101.6)
- added D68: LED, LED_SMD:LED_1206_3216Metric_Pad1.42x1.75mm_HandSolder, F.Cu at (144.7, 101.6)
- added D69: LED, LED_SMD:LED_1206_3216Metric_Pad1.42x1.75mm_HandSolder, F.Cu at (163.6, 101.6)
- added D70: LED, LED_SMD:LED_1206_3216Metric_Pad1.42x1.75mm_HandSolder, F.Cu at (182.7, 101.6)
- added D71: LED, LED_SMD:LED_1206_3216Metric_Pad1.42x1.75mm_HandSolder, F.Cu at (201.7, 101.6)
- added D72: LED, LED_SMD:LED_1206_3216Metric_Pad1.42x1.75mm_HandSolder, F.Cu at (220.7, 101.6)
- added D73: LED, LED_SMD:LED_1206_3216Metric_Pad1.42x1.75mm_HandSolder, F.Cu at (246.8, 101.6)
- added D74: LED, LED_SMD:LED_1206_3216Metric_Pad1.42x1.75mm_HandSolder, F.Cu at (33.0, 120.9)
- added D75: LED, LED_SMD:LED_1206_3216Metric_Pad1.42x1.75mm_HandSolder, F.Cu at (59.0, 120.7)
- added D76: LED, LED_SMD:LED_1206_3216Metric_Pad1.42x1.75mm_HandSolder, F.Cu at (78.1, 120.6)
- added D77: LED, LED_SMD:LED_1206_3216Metric_Pad1.42x1.75mm_HandSolder, F.Cu at (97.1, 120.7)
- added D78: LED, LED_SMD:LED_1206_3216Metric_Pad1.42x1.75mm_HandSolder, F.Cu at (116.3, 120.7)
- added D79: LED, LED_SMD:LED_1206_3216Metric_Pad1.42x1.75mm_HandSolder, F.Cu at (135.1, 120.6)
- added D80: LED, LED_SMD:LED_1206_3216Metric_Pad1.42x1.75mm_HandSolder, F.Cu at (154.3, 120.5)
- added D81: LED, LED_SMD:LED_1206_3216Metric_Pad1.42x1.75mm_HandSolder, F.Cu at (173.1, 120.5)
- added D82: LED, LED_SMD:LED_1206_3216Metric_Pad1.42x1.75mm_HandSolder, F.Cu at (192.2, 120.5)
- added D83: LED, LED_SMD:LED_1206_3216Metric_Pad1.42x1.75mm_HandSolder, F.Cu at (211.3, 120.5)
- added D84: LED, LED_SMD:LED_1206_3216Metric_Pad1.42x1.75mm_HandSolder, F.Cu at (230.2, 120.5)
- added D85: LED, LED_SMD:LED_1206_3216Metric_Pad1.42x1.75mm_HandSolder, F.Cu at (251.5, 120.6)
- added D86: LED, LED_SMD:LED_1206_3216Metric_Pad1.42x1.75mm_HandSolder, F.Cu at (28.3, 139.9)
- added D87: LED, LED_SMD:LED_1206_3216Metric_Pad1.42x1.75mm_HandSolder, F.Cu at (49.5, 139.9)
- added D88: LED, LED_SMD:LED_1206_3216Metric_Pad1.42x1.75mm_HandSolder, F.Cu at (71.0, 139.9)
- added D89: LED, LED_SMD:LED_1206_3216Metric_Pad1.42x1.75mm_HandSolder, F.Cu at (94.8, 139.9)
- added D90: LED, LED_SMD:LED_1206_3216Metric_Pad1.42x1.75mm_HandSolder, F.Cu at (123.3, 139.9)
- added D91: LED, LED_SMD:LED_1206_3216Metric_Pad1.42x1.75mm_HandSolder, F.Cu at (156.6, 139.9)
- added D92: LED, LED_SMD:LED_1206_3216Metric_Pad1.42x1.75mm_HandSolder, F.Cu at (185.0, 139.9)
- added D93: LED, LED_SMD:LED_1206_3216Metric_Pad1.42x1.75mm_HandSolder, F.Cu at (208.7, 139.8)
- added D94: LED, LED_SMD:LED_1206_3216Metric_Pad1.42x1.75mm_HandSolder, F.Cu at (230.2, 139.7)
- added J1: 2171790001, Library:MOLEX_2171790001, F.Cu at (272.2, 71.7)
- added J3: RESET, Jumper:SolderJumper-2_P1.3mm_Open_Pad1.0x1.5mm, F.Cu at (267.9, 96.6)
- added J4: HWB, Jumper:SolderJumper-2_P1.3mm_Open_Pad1.0x1.5mm, F.Cu at (267.9, 93.9)
- added J5: LED_ENABLE_JUMPER, Jumper:SolderJumper-2_P1.3mm_Open_Pad1.0x1.5mm, B.Cu at (264.1, 120.2)
- added R1: 511, Resistor_SMD:R_1206_3216Metric_Pad1.30x1.75mm_HandSolder, B.Cu at (257.6, 139.6)
- added R10: 511, Resistor_SMD:R_1206_3216Metric_Pad1.30x1.75mm_HandSolder, B.Cu at (183.9, 82.6)
- added R11: 511, Resistor_SMD:R_1206_3216Metric_Pad1.30x1.75mm_HandSolder, B.Cu at (202.9, 82.6)
- added R12: 511, Resistor_SMD:R_1206_3216Metric_Pad1.30x1.75mm_HandSolder, B.Cu at (222.1, 82.5)
- added R13: 511, Resistor_SMD:R_1206_3216Metric_Pad1.30x1.75mm_HandSolder, B.Cu at (240.7, 82.6)
- added R14: 511, Resistor_SMD:R_1206_3216Metric_Pad1.30x1.75mm_HandSolder, B.Cu at (259.1, 82.6)
- added R15: 511, Resistor_SMD:R_1206_3216Metric_Pad1.30x1.75mm_HandSolder, B.Cu at (33.8, 101.6)
- added R2: 511, Resistor_SMD:R_1206_3216Metric_Pad1.30x1.75mm_HandSolder, B.Cu at (31.6, 82.5)
- added R20: 511, Resistor_SMD:R_1206_3216Metric_Pad1.30x1.75mm_HandSolder, B.Cu at (55.9, 101.6)
- added R21: 511, Resistor_SMD:R_1206_3216Metric_Pad1.30x1.75mm_HandSolder, B.Cu at (74.5, 101.6)
- added R22: 511, Resistor_SMD:R_1206_3216Metric_Pad1.30x1.75mm_HandSolder, B.Cu at (93.7, 101.6)
- added R23: 511, Resistor_SMD:R_1206_3216Metric_Pad1.30x1.75mm_HandSolder, B.Cu at (112.8, 101.6)
- added R24: 511, Resistor_SMD:R_1206_3216Metric_Pad1.30x1.75mm_HandSolder, B.Cu at (131.8, 101.6)
- added R25: 511, Resistor_SMD:R_1206_3216Metric_Pad1.30x1.75mm_HandSolder, B.Cu at (150.9, 101.6)
- added R26: 511, Resistor_SMD:R_1206_3216Metric_Pad1.30x1.75mm_HandSolder, B.Cu at (169.6, 101.6)
- added R27: 511, Resistor_SMD:R_1206_3216Metric_Pad1.30x1.75mm_HandSolder, B.Cu at (188.8, 101.6)
- added R28: 511, Resistor_SMD:R_1206_3216Metric_Pad1.30x1.75mm_HandSolder, B.Cu at (207.8, 101.5)
- added R29: 511, Resistor_SMD:R_1206_3216Metric_Pad1.30x1.75mm_HandSolder, B.Cu at (227.1, 101.6)
- added R3: 511, Resistor_SMD:R_1206_3216Metric_Pad1.30x1.75mm_HandSolder, B.Cu at (50.5, 82.5)
- added R30: 511, Resistor_SMD:R_1206_3216Metric_Pad1.30x1.75mm_HandSolder, B.Cu at (252.7, 101.7)
- added R31: 511, Resistor_SMD:R_1206_3216Metric_Pad1.30x1.75mm_HandSolder, B.Cu at (39.1, 120.9)
- added R32: 511, Resistor_SMD:R_1206_3216Metric_Pad1.30x1.75mm_HandSolder, B.Cu at (65.0, 120.7)
- added R33: 511, Resistor_SMD:R_1206_3216Metric_Pad1.30x1.75mm_HandSolder, B.Cu at (84.0, 120.6)
- added R34: 511, Resistor_SMD:R_1206_3216Metric_Pad1.30x1.75mm_HandSolder, B.Cu at (102.8, 120.7)
- added R35: 511, Resistor_SMD:R_1206_3216Metric_Pad1.30x1.75mm_HandSolder, B.Cu at (122.2, 120.7)
- added R36: 511, Resistor_SMD:R_1206_3216Metric_Pad1.30x1.75mm_HandSolder, B.Cu at (141.1, 120.6)
- added R37: 511, Resistor_SMD:R_1206_3216Metric_Pad1.30x1.75mm_HandSolder, B.Cu at (160.2, 120.5)
- added R38: 511, Resistor_SMD:R_1206_3216Metric_Pad1.30x1.75mm_HandSolder, B.Cu at (179.1, 120.5)
- added R39: 511, Resistor_SMD:R_1206_3216Metric_Pad1.30x1.75mm_HandSolder, B.Cu at (198.2, 120.5)
- added R4: 511, Resistor_SMD:R_1206_3216Metric_Pad1.30x1.75mm_HandSolder, B.Cu at (69.8, 82.6)
- added R40: 511, Resistor_SMD:R_1206_3216Metric_Pad1.30x1.75mm_HandSolder, B.Cu at (217.4, 120.7)
- added R41: 511, Resistor_SMD:R_1206_3216Metric_Pad1.30x1.75mm_HandSolder, B.Cu at (236.2, 120.5)
- added R42: 511, Resistor_SMD:R_1206_3216Metric_Pad1.30x1.75mm_HandSolder, B.Cu at (257.4, 120.6)
- added R43: 511, Resistor_SMD:R_1206_3216Metric_Pad1.30x1.75mm_HandSolder, B.Cu at (34.1, 139.9)
- added R44: 511, Resistor_SMD:R_1206_3216Metric_Pad1.30x1.75mm_HandSolder, B.Cu at (55.5, 139.9)
- added R45: 511, Resistor_SMD:R_1206_3216Metric_Pad1.30x1.75mm_HandSolder, B.Cu at (77.0, 139.9)
- added R46: 511, Resistor_SMD:R_1206_3216Metric_Pad1.30x1.75mm_HandSolder, B.Cu at (100.8, 139.9)
- added R47: 511, Resistor_SMD:R_1206_3216Metric_Pad1.30x1.75mm_HandSolder, B.Cu at (129.3, 139.9)
- added R48: 511, Resistor_SMD:R_1206_3216Metric_Pad1.30x1.75mm_HandSolder, B.Cu at (162.8, 139.9)
- added R49: 511, Resistor_SMD:R_1206_3216Metric_Pad1.30x1.75mm_HandSolder, B.Cu at (191.1, 139.9)
- added R5: 511, Resistor_SMD:R_1206_3216Metric_Pad1.30x1.75mm_HandSolder, B.Cu at (89.0, 82.5)
- added R50: 511, Resistor_SMD:R_1206_3216Metric_Pad1.30x1.75mm_HandSolder, B.Cu at (214.7, 139.9)
- added R51: 511, Resistor_SMD:R_1206_3216Metric_Pad1.30x1.75mm_HandSolder, B.Cu at (236.2, 139.7)
- added R6: 511, Resistor_SMD:R_1206_3216Metric_Pad1.30x1.75mm_HandSolder, B.Cu at (107.8, 82.5)
- added R7: 511, Resistor_SMD:R_1206_3216Metric_Pad1.30x1.75mm_HandSolder, B.Cu at (127.0, 82.5)
- added R8: 511, Resistor_SMD:R_1206_3216Metric_Pad1.30x1.75mm_HandSolder, B.Cu at (146.1, 82.6)
- added R9: 511, Resistor_SMD:R_1206_3216Metric_Pad1.30x1.75mm_HandSolder, B.Cu at (165.1, 82.5)
- added REF**: MountingHole_2.2mm_M2, MountingHole:MountingHole_2.2mm_M2, F.Cu at (168.3, 86.4)
- added REF**: MountingHole_2.2mm_M2, MountingHole:MountingHole_2.2mm_M2, F.Cu at (45.9, 112.7)
- added REF**: MountingHole_2.2mm_M2, MountingHole:MountingHole_2.2mm_M2, F.Cu at (138.2, 133.1)
- added REF**: MountingHole_2.2mm_M2, MountingHole:MountingHole_2.2mm_M2, F.Cu at (78.2, 93.3)
- added REF**: MountingHole_2.2mm_M2, MountingHole:MountingHole_2.2mm_M2, F.Cu at (19.8, 111.5)
- added REF**: MountingHole_2.2mm_M2, MountingHole:MountingHole_2.2mm_M2, F.Cu at (241.6, 113.9)
- added REF**: MountingHole_2.2mm_M2, MountingHole:MountingHole_2.2mm_M2, F.Cu at (148.3, 106.4)
- added REF**: MountingHole_2.2mm_M2, MountingHole:MountingHole_2.2mm_M2, F.Cu at (83.2, 134.4)
- added REF**: MountingHole_2.2mm_M2, MountingHole:MountingHole_2.2mm_M2, F.Cu at (35.2, 71.0)
- added REF**: MountingHole_2.2mm_M2, MountingHole:MountingHole_2.2mm_M2, F.Cu at (266.1, 79.5)
- added REF**: MountingHole_2.2mm_M2, MountingHole:MountingHole_2.2mm_M2, F.Cu at (264.6, 132.8)
- C2: value EEE-HB1E4R7R -> 4.7uF; footprint Library:CAP_EEEFK1H220P -> Capacitor_SMD:C_1206_3216Metric_Pad1.33x1.80mm_HandSolder; moved to F.Cu
- D50: value D -> LED; footprint Diode_SMD:D_SOD-123 -> LED_SMD:LED_1206_3216Metric_Pad1.42x1.75mm_HandSolder; moved to F.Cu
- R16, R17, U1: moved to F.Cu
- R18, R19: value RMCF1206JT5K10 -> 5.1k; moved to F.Cu
- moved R19 120.2 mm to (275.4, 85.2), turned to -90 degrees
- moved C2 113.4 mm to (265.4, 71.9)
- moved U1 110.7 mm to (273.9, 138.8), turned to -90 degrees
- moved R18 109.5 mm to (267.3, 85.3), turned to -90 degrees
- moved C6 96.2 mm to (269.0, 108.2), turned to -90 degrees
- moved Y1 95.8 mm to (273.4, 112.5), turned to -90 degrees
- moved C5 90.4 mm to (269.0, 115.1), turned to 90 degrees
- moved C7 79.5 mm to (275.3, 93.6), turned to 90 degrees
- moved R17 73.3 mm to (272.8, 85.2), turned to -90 degrees
- moved R16 69.8 mm to (269.9, 85.2), turned to -90 degrees
- moved U2 60.7 mm to (265.5, 95.1)
- moved D50 9.12 mm to (251.6, 139.7), turned to 0 degrees
- moved D14 8.76 mm to (27.1, 90.2)
- moved D27 8.39 mm to (58.1, 109.2)
- moved D26 8.34 mm to (32.0, 109.5)
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Connections:
- D50 pad 1: ROW_4 -> GND
- D50 pad 2: /Matrix/D_C12R4 -> Net-(D50-A)
Routing:
- net GND: track 0.00 -> 1340.5 mm, vias 0 -> 35
- net /LED Circuit/LED_5V: track 0.00 -> 1011.7 mm, vias 0 -> 8
- net COL_1: track 0.00 -> 353.6 mm
- net COL_2: track 0.00 -> 321.6 mm, vias 0 -> 3
- net COL_3: track 0.00 -> 298.6 mm, vias 0 -> 5
- net ROW_4: track 0.00 -> 297.9 mm, vias 0 -> 6
- net ROW_1: track 0.00 -> 282.8 mm
- net ROW_3: track 0.00 -> 271.4 mm
- net COL_4: track 0.00 -> 257.2 mm, vias 0 -> 4
- net ROW_2: track 0.00 -> 244.1 mm
- net COL_5: track 0.00 -> 242.2 mm, vias 0 -> 6
- net COL_6: track 0.00 -> 220.8 mm, vias 0 -> 6
- net COL_7: track 0.00 -> 205.6 mm, vias 0 -> 7
- net COL_8: track 0.00 -> 191.7 mm, vias 0 -> 5
- net COL_9: track 0.00 -> 164.8 mm, vias 0 -> 10
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- added copper zone on B.Cu, net GND
- added copper zone on F.Cu, net GND
Other:
- board size 247 x 91.2 mm -> 261.1 x 76.2 mm
- board text added: "Designed by Luke Zambella"
- board text removed: "${REFERENCE}"
- board text removed: "Designed by Luke Zambella Rev2"
- board text removed: "MCU"
