File: schematics/rev2/40 Keyboard.kicad_sch (KiCad schematic)
At the start: 7 parts, among them J2 2171790001

Commit message: Update key layout, increase debounce, PCB update
Parts:
- removed C1: C3216X7R2A334K130AA, Capacitor_SMD:C_1206_3216Metric, symbol Project:EEEFK1H220P
- removed D48: LED, LED_THT:LED_D3.0mm, symbol Device:LED
- removed R15: 1k, Resistor_SMD:R_1206_3216Metric, symbol Device:R
Other:
- moved on the sheet: C2, J2, R18, R19

Commit message: Update schematic and board layout
Parts:
- C2: value EEE-HB1E4R7R -> 4.7uF; footprint Library:CAP_EEEFK1H220P -> Capacitor_SMD:C_1206_3216Metric_Pad1.33x1.80mm_HandSolder
- J1: renamed from J2; Part # (none) -> 2171790001
- R18, R19: value RMCF1206JT5K10 -> 5.1k; Part # (none) -> RMCF1206JT5K10
Other:
- added sheet LED Circuit (untitled.kicad_sch)
